File: Digispark USB.kicad_sch (KiCad schematic)
At the start: 12 parts, among them J1 Conn_01x04, J2 Conn_01x04, U2 ATtiny85-20S

Commit message: pdfs
Other:
- company: (none) -> SoloScriptSage - Vladyslav Hirchuk
- title: (none) -> Digispark USB Development Board
- moved on the sheet: R2
